Commit message: Updated car measurements

File: opponent_racecar.xacro (robot description, xacro)
@@ -2,10 +2,10 @@
 <!-- A simple model of the racecar for rviz -->
 <robot xmlns:xacro="http://www.ros.org/wiki/xacro" name="opponent_racecar">
-  <xacro:property name="wheelbase" value="0.325" />
-  <xacro:property name="width" value="0.2" />
+  <xacro:property name="wheelbase" value="0.3302" />
+  <xacro:property name="width" value="0.2032" />
   <xacro:property name="height" value="0.1" />
   <xacro:property name="ground_offset" value="0.04" />
-  <xacro:property name="wheel_radius" value="0.05" />
-  <xacro:property name="wheel_length" value="0.045" />
+  <xacro:property name="wheel_radius" value="0.0508" />
+  <xacro:property name="wheel_length" value="0.0381" />
   <xacro:property name="laser_distance_from_base_link" value="0.275" />
   <xacro:property name="laser_height" value="0.05" />
