Commit message: Updated depencies, made measurements match real racecar and added laser to model

File: racecar.xacro (robot description, xacro)
@@ -2,12 +2,18 @@
 <!-- A simple model of the racecar for rviz -->
 <robot xmlns:xacro="http://www.ros.org/wiki/xacro" name="racecar">
-	<xacro:property name="wheelbase" value="0.34" />
+	<xacro:property name="wheelbase" value="0.325" />
 	<xacro:property name="width" value="0.2" />
 	<xacro:property name="height" value="0.1" />
-  <xacro:property name="ground_offset" value="0.03" />
+  <xacro:property name="ground_offset" value="0.04" />
   <xacro:property name="wheel_radius" value="0.05" />
-	<xacro:property name="wheel_length" value="0.03" />
+	<xacro:property name="wheel_length" value="0.045" />
+	<xacro:property name="laser_distance_from_base_link" value="0.275" />
+	<xacro:property name="laser_height" value="0.05" />
+	<xacro:property name="laser_radius" value="0.026" />
+  <material name="black">
+    <color rgba="0.2 0.2 0.2 1."/>
+  </material>
   <material name="blue">
-    <color rgba="0. 0. 0.8 1."/>
+    <color rgba="0.3 0.57 1. 1."/>
   </material>
 	<link name="base_link">
@@ -18,4 +24,17 @@
 			</geometry>
       <material name="blue"/>
+		</visual>
+	</link>
+	<joint name="base_to_laser_model" type="fixed">
+		<parent link="base_link"/>
+		<child link="laser_model"/>
+		<origin xyz="${laser_distance_from_base_link} 0 ${ground_offset+height+(laser_height/2)}"/>
+	</joint>
+	<link name="laser_model">
+		<visual>
+			<geometry>
+				<cylinder radius="${laser_radius}" length="${laser_height}"/>
+			</geometry>
+      <material name="black"/>
 		</visual>
 	</link>
@@ -30,4 +49,5 @@
 				<cylinder radius="${wheel_radius}" length="${wheel_length}"/>
 			</geometry>
+      <material name="black"/>
       <origin rpy="${pi/2} 0 0"/>
 		</visual>
@@ -43,4 +63,5 @@
 				<cylinder radius="${wheel_radius}" length="${wheel_length}"/>
 			</geometry>
+      <material name="black"/>
       <origin rpy="${pi/2} 0 0"/>
 		</visual>
@@ -61,4 +82,5 @@
 				<cylinder radius="${wheel_radius}" length="${wheel_length}"/>
 			</geometry>
+      <material name="black"/>
       <origin rpy="${pi/2} 0 0"/>
 		</visual>
@@ -79,4 +101,5 @@
 				<cylinder radius="${wheel_radius}" length="${wheel_length}"/>
 			</geometry>
+      <material name="black"/>
       <origin rpy="${pi/2} 0 0"/>
 		</visual>

Commit message: Updated documentation

File: racecar.xacro (robot description, xacro)
@@ -2,13 +2,13 @@
 <!-- A simple model of the racecar for rviz -->
 <robot xmlns:xacro="http://www.ros.org/wiki/xacro" name="racecar">
-	<xacro:property name="wheelbase" value="0.325" />
-	<xacro:property name="width" value="0.2" />
-	<xacro:property name="height" value="0.1" />
+  <xacro:property name="wheelbase" value="0.325" />
+  <xacro:property name="width" value="0.2" />
+  <xacro:property name="height" value="0.1" />
   <xacro:property name="ground_offset" value="0.04" />
   <xacro:property name="wheel_radius" value="0.05" />
-	<xacro:property name="wheel_length" value="0.045" />
-	<xacro:property name="laser_distance_from_base_link" value="0.275" />
-	<xacro:property name="laser_height" value="0.05" />
-	<xacro:property name="laser_radius" value="0.026" />
+  <xacro:property name="wheel_length" value="0.045" />
+  <xacro:property name="laser_distance_from_base_link" value="0.275" />
+  <xacro:property name="laser_height" value="0.05" />
+  <xacro:property name="laser_radius" value="0.026" />
   <material name="black">
     <color rgba="0.2 0.2 0.2 1."/>
@@ -17,59 +17,59 @@
     <color rgba="0.3 0.57 1. 1."/>
   </material>
-	<link name="base_link">
-		<visual>
+  <link name="base_link">
+    <visual>
       <origin xyz="${wheelbase/2} 0 ${ground_offset+height/2}"/>
-			<geometry>
+      <geometry>
         <box size="${wheelbase} ${width} ${height}"/>
-			</geometry>
+      </geometry>
       <material name="blue"/>
-		</visual>
-	</link>
-	<joint name="base_to_laser_model" type="fixed">
-		<parent link="base_link"/>
-		<child link="laser_model"/>
-		<origin xyz="${laser_distance_from_base_link} 0 ${ground_offset+height+(laser_height/2)}"/>
-	</joint>
-	<link name="laser_model">
-		<visual>
-			<geometry>
-				<cylinder radius="${laser_radius}" length="${laser_height}"/>
-			</geometry>
+    </visual>
+  </link>
+  <joint name="base_to_laser_model" type="fixed">
+    <parent link="base_link"/>
+    <child link="laser_model"/>
+    <origin xyz="${laser_distance_from_base_link} 0 ${ground_offset+height+(laser_height/2)}"/>
+  </joint>
+  <link name="laser_model">
+    <visual>
+      <geometry>
+        <cylinder radius="${laser_radius}" length="${laser_height}"/>
+      </geometry>
       <material name="black"/>
-		</visual>
-	</link>
-	<joint name="base_to_back_left_wheel" type="fixed">
-		<parent link="base_link"/>
-		<child link="back_left_wheel"/>
+    </visual>
+  </link>
+  <joint name="base_to_back_left_wheel" type="fixed">
+    <parent link="base_link"/>
+    <child link="back_left_wheel"/>
     <origin xyz="0 ${(wheel_length+width)/2} ${wheel_radius}"/>
-	</joint>
-	<link name="back_left_wheel">
-		<visual>
-			<geometry>
-				<cylinder radius="${wheel_radius}" length="${wheel_length}"/>
-			</geometry>
+  </joint>
+  <link name="back_left_wheel">
+    <visual>
+      <geometry>
+        <cylinder radius="${wheel_radius}" length="${wheel_length}"/>
+      </geometry>
       <material name="black"/>
       <origin rpy="${pi/2} 0 0"/>
-		</visual>
-	</link>
-	<joint name="base_to_back_right_wheel" type="fixed">
-		<parent link="base_link"/>
-		<child link="back_right_wheel"/>
+    </visual>
+  </link>
+  <joint name="base_to_back_right_wheel" type="fixed">
+    <parent link="base_link"/>
+    <child link="back_right_wheel"/>
     <origin xyz="0 ${-(wheel_length+width)/2} ${wheel_radius}"/>
-	</joint>
-	<link name="back_right_wheel">
-		<visual>
-			<geometry>
-				<cylinder radius="${wheel_radius}" length="${wheel_length}"/>
-			</geometry>
+  </joint>
+  <link name="back_right_wheel">
+    <visual>
+      <geometry>
+        <cylinder radius="${wheel_radius}" length="${wheel_length}"/>
+      </geometry>
       <material name="black"/>
       <origin rpy="${pi/2} 0 0"/>
-		</visual>
-	</link>
-	<joint name="base_to_front_left_hinge" type="fixed">
-		<parent link="base_link"/>
-		<child link="front_left_hinge"/>
+    </visual>
+  </link>
+  <joint name="base_to_front_left_hinge" type="fixed">
+    <parent link="base_link"/>
+    <child link="front_left_hinge"/>
     <origin xyz="${wheelbase} ${(wheel_length+width)/2} ${wheel_radius}"/>
-	</joint>
+  </joint>
   <link name="front_left_hinge"/>
   <joint name="front_left_hinge_to_wheel" type="continuous">
@@ -77,18 +77,18 @@
     <child link="front_left_wheel"/>
   </joint>
-	<link name="front_left_wheel">
-		<visual>
-			<geometry>
-				<cylinder radius="${wheel_radius}" length="${wheel_length}"/>
-			</geometry>
+  <link name="front_left_wheel">
+    <visual>
+      <geometry>
+        <cylinder radius="${wheel_radius}" length="${wheel_length}"/>
+      </geometry>
       <material name="black"/>
       <origin rpy="${pi/2} 0 0"/>
-		</visual>
-	</link>
-	<joint name="base_to_front_right_hinge" type="fixed">
-		<parent link="base_link"/>
-		<child link="front_right_hinge"/>
+    </visual>
+  </link>
+  <joint name="base_to_front_right_hinge" type="fixed">
+    <parent link="base_link"/>
+    <child link="front_right_hinge"/>
     <origin xyz="${wheelbase} ${-(wheel_length+width)/2} ${wheel_radius}"/>
-	</joint>
+  </joint>
   <link name="front_right_hinge"/>
   <joint name="front_right_hinge_to_wheel" type="continuous">
@@ -96,12 +96,12 @@
     <child link="front_right_wheel"/>
   </joint>
-	<link name="front_right_wheel">
-		<visual>
-			<geometry>
-				<cylinder radius="${wheel_radius}" length="${wheel_length}"/>
-			</geometry>
+  <link name="front_right_wheel">
+    <visual>
+      <geometry>
+        <cylinder radius="${wheel_radius}" length="${wheel_length}"/>
+      </geometry>
       <material name="black"/>
       <origin rpy="${pi/2} 0 0"/>
-		</visual>
-	</link>
+    </visual>
+  </link>
 </robot>

Commit message: New branch

File: racecar.xacro (robot description, xacro)
@@ -2,10 +2,10 @@
 <!-- A simple model of the racecar for rviz -->
 <robot xmlns:xacro="http://www.ros.org/wiki/xacro" name="racecar">
-  <xacro:property name="wheelbase" value="0.325" />
-  <xacro:property name="width" value="0.2" />
+  <xacro:property name="wheelbase" value="0.3302" />
+  <xacro:property name="width" value="0.2032" />
   <xacro:property name="height" value="0.1" />
   <xacro:property name="ground_offset" value="0.04" />
-  <xacro:property name="wheel_radius" value="0.05" />
-  <xacro:property name="wheel_length" value="0.045" />
+  <xacro:property name="wheel_radius" value="0.0508" />
+  <xacro:property name="wheel_length" value="0.0381" />
   <xacro:property name="laser_distance_from_base_link" value="0.275" />
   <xacro:property name="laser_height" value="0.05" />

Commit message: use the robot model from racecar_description

File: racecar.xacro (robot description, xacro)
@@ -39,10 +39,10 @@
     </visual>
   </link>
-  <joint name="base_to_back_left_wheel" type="fixed">
+  <joint name="base_to_left_rear_wheel" type="fixed">
     <parent link="base_link"/>
-    <child link="back_left_wheel"/>
+    <child link="left_rear_wheel"/>
     <origin xyz="0 ${(wheel_length+width)/2} ${wheel_radius}"/>
   </joint>
-  <link name="back_left_wheel">
+  <link name="left_rear_wheel">
     <visual>
       <geometry>
@@ -53,10 +53,10 @@
     </visual>
   </link>
-  <joint name="base_to_back_right_wheel" type="fixed">
+  <joint name="base_to_right_rear_wheel" type="fixed">
     <parent link="base_link"/>
-    <child link="back_right_wheel"/>
+    <child link="right_rear_wheel"/>
     <origin xyz="0 ${-(wheel_length+width)/2} ${wheel_radius}"/>
   </joint>
-  <link name="back_right_wheel">
+  <link name="right_rear_wheel">
     <visual>
       <geometry>
@@ -67,15 +67,15 @@
     </visual>
   </link>
-  <joint name="base_to_front_left_hinge" type="fixed">
+  <joint name="base_to_left_steering_hinge" type="fixed">
     <parent link="base_link"/>
-    <child link="front_left_hinge"/>
+    <child link="left_steering_hinge"/>
     <origin xyz="${wheelbase} ${(wheel_length+width)/2} ${wheel_radius}"/>
   </joint>
-  <link name="front_left_hinge"/>
-  <joint name="front_left_hinge_to_wheel" type="continuous">
-    <parent link="front_left_hinge"/>
-    <child link="front_left_wheel"/>
+  <link name="left_steering_hinge"/>
+  <joint name="left_steering_hinge_to_wheel" type="continuous">
+    <parent link="left_steering_hinge"/>
+    <child link="left_front_wheel"/>
   </joint>
-  <link name="front_left_wheel">
+  <link name="left_front_wheel">
     <visual>
       <geometry>
@@ -86,15 +86,15 @@
     </visual>
   </link>
-  <joint name="base_to_front_right_hinge" type="fixed">
+  <joint name="base_to_right_steering_hinge" type="fixed">
     <parent link="base_link"/>
-    <child link="front_right_hinge"/>
+    <child link="right_steering_hinge"/>
     <origin xyz="${wheelbase} ${-(wheel_length+width)/2} ${wheel_radius}"/>
   </joint>
-  <link name="front_right_hinge"/>
-  <joint name="front_right_hinge_to_wheel" type="continuous">
-    <parent link="front_right_hinge"/>
-    <child link="front_right_wheel"/>
+  <link name="right_steering_hinge"/>
+  <joint name="right_steering_hinge_to_wheel" type="continuous">
+    <parent link="right_steering_hinge"/>
+    <child link="right_front_wheel"/>
   </joint>
-  <link name="front_right_wheel">
+  <link name="right_front_wheel">
     <visual>
       <geometry>
